File: WeMos-Lora.sch (EAGLE design)
At the start: 20 parts, among them P1 PADNORMAL, P2 PADNORMAL, P3 PADNORMAL, P4 PADNORMAL

Commit message: Version V1.1
- OLED Display connector has now lock pad
- Antenna signal with via all around
- ground plane set to 12min blocking to avoid short circuit with
connectors in rarely cases
- Added footprint for Microchip 24AA02E64 64 bits serial number
Parts:
- removed J$1: ANTENNASMALL, _c2h:ANTENNASMALL
- added C5: 100nF, _c2h:CAP0805-CAP
- added D2, D3, D4: 1N4148, Seeed-Discrete:D-ESD-2P-CESD5V0D1
- added J$2: ANTENNATINY, _c2h:ANTENNATINY
- added U1: 24AA02E64T, Microchip-24AA02E64T:24AA02E64T-I/OT
- I2C_OLED: value CON_HEADER_1X04'SMALL'' -> CON_HEADER_1X04'LOCK'; device _c2h:CON_HEADER_1X04'SMALL'' -> _c2h:CON_HEADER_1X04'LOCK'
Connections:
- new net DIO0: D2.1, U$5.DIO0
- new net DIO1: D3.1, U$5.DIO1
- new net DIO2: D4.1, U$5.DIO2
- net 3V3: now also C5.1, U1.VCC
- net ANT: now also J$2.SIGNAL; no longer J$1.SIGNAL
- net GND: now also C5.2, J$2.GND@0, J$2.GND@1, J$2.GND@2, J$2.GND@3, U1.VSS; no longer J$1.GND@0, J$1.GND@1, J$1.GND@2, J$1.GND@3
- net GPIO15: now also D2.2, D3.2, D4.2; no longer U$5.DIO0
- net RST: now also U$5.RST
- net SCL: now also U1.SCL
- net SDA: now also U1.SDA
Other:
- note added: "FLASH/RGBLED"
- note added: "Switch"
- note added: "WeMos already has a pulldown on GPIO15"
- note removed: "FLASH"

Commit message: Bump to V1.2
Parts:
- added JP3: DS, _c2h:JUMPER-PAD-3-2OF3_NC_BY_TRACE_SMALL
- added R3: 100K, _c2h:RESISTOR0805-RES
Connections:
- new net SEL: JP3.3, R3.2, U$5.SEL
- net GND: now also R3.1
- net GPIO16: now also JP3.2; no longer U$5.SEL
- net RST: now also JP3.1
Other:
- note added: "868MHz"
- note added: "WeMos has a 12K pulldown on GPIO15"
- note added: "WeMos has a 12K pullup on GPIO2"
- note removed: "433MHz"
- note removed: "WeMos already has a pulldown on GPIO15"
- note removed: "WeMos already has a pullup on GPIO2"
Changed lines of the file:
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@@
 <?xml version="1.0" encoding="utf-8"?>
 <!DOCTYPE eagle SYSTEM "eagle.dtd">
-<eagle version="7.6.0">
+<eagle version="7.7.0">
 <drawing>
 <settings>
@@
 <part name="NAME" library="SparkFun-Aesthetics" deviceset="FRAME-A4L" device="" value="Value">
 <attribute name="CNAME" value="ESP8266 WeMos Lora Shield"/>
-<attribute name="CREVISION" value="1.1"/>
+<attribute name="CREVISION" value="1.2"/>
 <attribute name="DESIGNER" value="Charles-Henri Hallard"/>
 </part>
@@
 <part name="C5" library="_c2h" deviceset="CAP" device="0805-CAP" value="100nF"/>
 <part name="GND7" library="SparkFun" deviceset="GND" device=""/>
+<part name="JP3" library="_c2h" deviceset="JUMPER-PAD-3-2OF3_NC_BY_TRACE" device="_SMALL" value="DS"/>
+<part name="R3" library="_c2h" deviceset="RESISTOR" device="0805-RES" value="100K"/>
+<part name="GND11" library="supply1" deviceset="GND" device=""/>
 </parts>
 <sheets>
@@
 <text x="134.62" y="125.73" size="1.778" layer="94">IRQ</text>
 <text x="153.67" y="146.05" size="2.54" layer="94">WeMos  Headers</text>
-<text x="99.06" y="123.19" size="1.778" layer="94">433MHz</text>
+<text x="99.06" y="123.19" size="1.778" layer="94">868MHz</text>
 <text x="191.77" y="128.27" size="1.778" layer="94">Switch</text>
 <text x="46.99" y="124.46" size="1.778" layer="94">SS</text>
@@
 <text x="44.45" y="119.38" size="1.778" layer="94">MISO</text>
 <text x="45.72" y="121.92" size="1.778" layer="94">SCK</text>
-<text x="119.38" y="92.71" size="1.778" layer="94">WeMos already has
-a pullup on GPIO2</text>
-<text x="134.62" y="135.89" size="1.778" layer="94">SS</text>
-<text x="111.76" y="45.72" size="1.778" layer="94">WeMos already
-has a pulldown
-on GPIO15</text>
+<text x="117.475" y="89.535" size="1.778" layer="94">WeMos  has a 12K
+pullup on GPIO2</text>
+<text x="109.855" y="49.53" size="1.778" layer="94">WeMos has a 12K
+pulldown on GPIO15</text>
+<text x="118.745" y="129.54" size="1.778" layer="94">SS</text>
 </plain>
 <instances>
@@
 <attribute name="VALUE" x="77.47" y="49.53" size="1.778" layer="96" rot="R90"/>
 </instance>
+<instance part="JP3" gate="G$1" x="128.27" y="135.89" rot="MR0"/>
+<instance part="R3" gate="G$1" x="123.825" y="123.19" smashed="yes" rot="R90">
+<attribute name="NAME" x="122.3264" y="121.92" size="1.778" layer="95" rot="R90"/>
+<attribute name="VALUE" x="127.127" y="120.65" size="1.778" layer="96" rot="R90"/>
+</instance>
+<instance part="GND11" gate="1" x="123.825" y="114.935"/>
 </instances>
 <busses>
@@
 <wire x1="71.12" y1="52.07" x2="72.39" y2="52.07" width="0.1524" layer="91"/>
 </segment>
+<segment>
+<pinref part="R3" gate="G$1" pin="1"/>
+<pinref part="GND11" gate="1" pin="GND"/>
+<wire x1="123.825" y1="118.11" x2="123.825" y2="117.475" width="0.1524" layer="91"/>
+</segment>
 </net>
 <net name="SCL" class="0">
@@
 <label x="52.07" y="114.3" size="1.778" layer="95"/>
 </segment>
+<segment>
+<pinref part="JP3" gate="G$1" pin="1"/>
+<wire x1="128.27" y1="140.97" x2="128.27" y2="142.24" width="0.1524" layer="91"/>
+<wire x1="128.27" y1="142.24" x2="118.11" y2="142.24" width="0.1524" layer="91"/>
+<label x="118.11" y="142.24" size="1.778" layer="95" rot="R180" xref="yes"/>
+</segment>
 </net>
 <net name="GPIO16" class="0">
 <segment>
 <pinref part="JP2" gate="G$1" pin="3"/>
-<wire x1="148.59" y1="135.89" x2="140.97" y2="135.89" width="0.1524" layer="91"/>
 <label x="140.97" y="135.89" size="1.778" layer="95"/>
-</segment>
-<segment>
-<wire x1="63.5" y1="124.46" x2="50.8" y2="124.46" width="0.1524" layer="91"/>
-<label x="52.07" y="124.46" size="1.778" layer="95"/>
-<pinref part="U$5" gate="G$1" pin="SEL"/>
-<junction x="63.5" y="124.46"/>
+<pinref part="JP3" gate="G$1" pin="2"/>
+<wire x1="148.59" y1="135.89" x2="133.35" y2="135.89" width="0.1524" layer="91"/>
 </segment>
 </net>
@@
 </segment>
 </net>
+<net name="SEL" class="0">
+<segment>
+<pinref part="JP3" gate="G$1" pin="3"/>
+<wire x1="128.27" y1="130.81" x2="128.27" y2="129.54" width="0.1524" layer="91"/>
+<wire x1="128.27" y1="129.54" x2="123.825" y2="129.54" width="0.1524" layer="91"/>
+<label x="118.11" y="129.54" size="1.778" layer="95" rot="R180" xref="yes"/>
+<pinref part="R3" gate="G$1" pin="2"/>
+<wire x1="123.825" y1="129.54" x2="118.11" y2="129.54" width="0.1524" layer="91"/>
+<wire x1="123.825" y1="128.27" x2="123.825" y2="129.54" width="0.1524" layer="91"/>
+<junction x="123.825" y="129.54"/>
+</segment>
+<segment>
+<wire x1="63.5" y1="124.46" x2="50.8" y2="124.46" width="0.1524" layer="91"/>
+<label x="52.07" y="124.46" size="1.778" layer="95"/>
+<pinref part="U$5" gate="G$1" pin="SEL"/>
+<junction x="63.5" y="124.46"/>
+</segment>
+</net>

Commit message: Bump to v1.3
Parts:
- added U$2: PAD-JUMPER-SWAPSWAP, _c2h:PAD-JUMPER-SWAPSWAP
Connections:
- new net 3V3_GD: I2C_OLED.1, U$2.3
- new net GD_3V3: I2C_OLED.2, U$2.2
- net 3V3: now also U$2.4; no longer I2C_OLED.1
- net GND: now also U$2.1; no longer I2C_OLED.2
